File: Electronics/_saved_Pads.sch (KiCad schematic (older format))
At the start: 7 parts, among them P1 Header, SW1 SW_PUSH, SW2 SW_PUSH, SW3 SW_PUSH, SW4 SW_PUSH

Commit message: created V1 of the pcb and SKQUAAA010 footprint
Parts:
- P1: footprint (none) -> Socket_Strips:Socket_Strip_Straight_1x10
- P2: renamed from P?; footprint (none) -> Socket_Strips:Socket_Strip_Straight_1x02
- SW1, SW2, SW3, SW4: footprint (none) -> Buttons_Switches_ThroughHole:SW_PUSH_6mm
- SW5: renamed from SW?; footprint (none) -> footprints:ALPS_SKQUAAA010
Changed lines of the file:
@@
 LIBS:valves
 LIBS:alps_skquaaa010
+LIBS:Pads-cache
 EELAYER 25 0
 EELAYER END
@@
 F 0 "P1" H 3200 2350 50  0000 C CNN
 F 1 "Header" V 3300 1800 50  0000 C CNN
-F 2 "" H 3200 1800 50  0000 C CNN
+F 2 "Socket_Strips:Socket_Strip_Straight_1x10" H 3200 1800 50  0001 C CNN
 F 3 "" H 3200 1800 50  0000 C CNN
 	1    3200 1800
@@
 F 0 "SW1" H 4350 2660 50  0000 C CNN
 F 1 "SW_PUSH" H 4200 2470 50  0000 C CNN
-F 2 "" H 4200 2550 50  0000 C CNN
+F 2 "Buttons_Switches_ThroughHole:SW_PUSH_6mm" H 4200 2550 50  0001 C CNN
 F 3 "" H 4200 2550 50  0000 C CNN
 	1    4200 2550
@@
 F 0 "SW2" H 4350 3010 50  0000 C CNN
 F 1 "SW_PUSH" H 4200 2820 50  0000 C CNN
-F 2 "" H 4200 2900 50  0000 C CNN
+F 2 "Buttons_Switches_ThroughHole:SW_PUSH_6mm" H 4200 2900 50  0001 C CNN
 F 3 "" H 4200 2900 50  0000 C CNN
 	1    4200 2900
@@
 F 0 "SW3" H 4350 3360 50  0000 C CNN
 F 1 "SW_PUSH" H 4200 3170 50  0000 C CNN
-F 2 "" H 4200 3250 50  0000 C CNN
+F 2 "Buttons_Switches_ThroughHole:SW_PUSH_6mm" H 4200 3250 50  0001 C CNN
 F 3 "" H 4200 3250 50  0000 C CNN
 	1    4200 3250
@@
 F 0 "SW4" H 4350 3710 50  0000 C CNN
 F 1 "SW_PUSH" H 4200 3520 50  0000 C CNN
-F 2 "" H 4200 3600 50  0000 C CNN
+F 2 "Buttons_Switches_ThroughHole:SW_PUSH_6mm" H 4200 3600 50  0001 C CNN
 F 3 "" H 4200 3600 50  0000 C CNN
 	1    4200 3600
@@
 $EndComp
 $Comp
-L GND #PWR1
+L GND #PWR01
 U 1 1 588B9DEE
 P 2750 2150
-F 0 "#PWR1" H 2750 1900 50  0001 C CNN
+F 0 "#PWR01" H 2750 1900 50  0001 C CNN
 F 1 "GND" H 2750 2000 50  0000 C CNN
 F 2 "" H 2750 2150 50  0000 C CNN
@@
 	2750 2000 2750 2150
 $Comp
-L GND #PWR2
+L GND #PWR02
 U 1 1 588B9ECD
 P 4900 3100
-F 0 "#PWR2" H 4900 2850 50  0001 C CNN
+F 0 "#PWR02" H 4900 2850 50  0001 C CNN
 F 1 "GND" H 4900 2950 50  0000 C CNN
 F 2 "" H 4900 3100 50  0000 C CNN
@@
 	3350 3600 3900 3600
 $Comp
-L ALPS_SKQUAAA010 SW?
+L ALPS_SKQUAAA010 SW5
 U 1 1 588BA1ED
 P 3100 3300
-F 0 "SW?" V 2800 2850 60  0000 C CNN
+F 0 "SW5" V 2800 2850 60  0000 C CNN
 F 1 "ALPS_SKQUAAA010" V 3100 3100 60  0000 C CNN
-F 2 "" H 3100 3300 60  0001 C CNN
+F 2 "footprints:ALPS_SKQUAAA010" H 3100 3300 60  0001 C CNN
 F 3 "" H 3100 3300 60  0001 C CNN
 	1    3100 3300
@@
 	2900 2600 2900 2800
 $Comp
-L CONN_01X02 P?
+L CONN_01X02 P2
 U 1 1 588BA38C
 P 1900 2700
-F 0 "P?" H 1900 2850 50  0000 C CNN
+F 0 "P2" H 1900 2850 50  0000 C CNN
 F 1 "CONN_01X02" V 2000 2700 50  0000 C CNN
-F 2 "" H 1900 2700 50  0000 C CNN
+F 2 "Socket_Strips:Socket_Strip_Straight_1x02" H 1900 2700 50  0001 C CNN
 F 3 "" H 1900 2700 50  0000 C CNN
 	1    1900 2700
@@
 	2850 2650 2100 2650
 $Comp
-L GND #PWR?
+L GND #PWR03
 U 1 1 588BA3ED
 P 2250 2800
-F 0 "#PWR?" H 2250 2550 50  0001 C CNN
+F 0 "#PWR03" H 2250 2550 50  0001 C CNN
 F 1 "GND" H 2250 2650 50  0000 C CNN
 F 2 "" H 2250 2800 50  0000 C CNN
@@
 	2250 2750 2250 2800
 $Comp
-L GND #PWR?
+L GND #PWR04
 U 1 1 588BA46C
 P 2350 3200
-F 0 "#PWR?" H 2350 2950 50  0001 C CNN
+F 0 "#PWR04" H 2350 2950 50  0001 C CNN
 F 1 "GND" H 2350 3050 50  0000 C CNN
 F 2 "" H 2350 3200 50  0000 C CNN
